File: PCB/Keypad.kicad_pcb (KiCad board)
At the start: 2 copper layers, 80.2 x 100 mm, 33 parts, among them SW1 RotaryEncoder_Switch, SW10 SW_Push, SW11 SW_Push, SW12 SW_Push, SW13 SW_Push, SW14 SW_Push, SW15 SW_Push, SW16 SW_Push, SW2 SW_Push, SW3 SW_Push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

Commit message: Add files via upload
Parts:
- moved D10 9.18 mm to (110.7, 119.2)
- moved D7 5.75 mm to (95.0, 79.9)
- moved D9 4.63 mm to (96.1, 118.5)
- moved D11 3.03 mm to (130.5, 118.7)
- moved D2 2.73 mm to (130.8, 99.7)
- moved D6 2.69 mm to (115.1, 80.2)
- moved D1 2.58 mm to (150.5, 100.2)
- moved D12 2.15 mm to (149.6, 118.5)
- moved D5 2.06 mm to (131.5, 81.0)
- moved D4 2.00 mm to (96.0, 100.0)
- moved D3 1.75 mm to (110.2, 99.5)
- moved D14 1.58 mm to (113.9, 137.0)
- moved D13 1.21 mm to (97.4, 137.2)
- moved D15 0.68 mm to (132.3, 136.9)
- moved D16 0.16 mm to (149.8, 137.6)
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Routing:
- net Net-(D10-K): track 106.7 -> 139.9 mm, vias 0 -> 1
- net Net-(U1-GPIO26/ADC0/A0): track 23.4 -> 0.00 mm
- net Net-(U1-GPIO1/RX): track 148.3 -> 129.7 mm
- net Net-(D13-K): track 131.8 -> 138.9 mm
- net Net-(D10-A): track 4.00 -> 10.7 mm
- net Net-(D5-K): track 58.9 -> 64.3 mm
- net Net-(U1-GPIO7/SCL): track 111.1 -> 106.6 mm
- net Net-(D7-A): track 11.2 -> 7.52 mm
- net Net-(D1-K): track 85.3 -> 88.7 mm
- net Net-(D11-A): track 7.27 -> 10.1 mm
- net Net-(D5-A): track 8.72 -> 6.53 mm
- net Net-(D12-A): track 7.95 -> 10.1 mm
- net Net-(D9-A): track 4.34 -> 6.46 mm
- net Net-(D1-A): track 8.38 -> 6.40 mm
- net Net-(D14-A): track 6.21 -> 7.89 mm
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